File: Drone_ESC_Bridge.kicad_pcb (KiCad board)
At the start: 2 copper layers, 52 x 33 mm, 21 parts, among them Q1 Si2318CDS, U1 LMP8640, U2 LM5050-1

Commit message: Initial board revision
Parts:
- moved SPI1 4.41 mm to (153.2, 129.6)
- moved C1 3.68 mm to (146.3, 130.9)
- moved JETSON_PWR1 3.67 mm to (143.8, 129.6)
- moved C4 3.66 mm to (138.7, 130.9)
- moved C5 3.47 mm to (132.5, 129.8)
- moved C3 1.35 mm to (120.5, 123.3)
- moved R2 1.19 mm to (120.4, 117.7)
- moved U2 1.19 mm to (120.4, 120.5)
- moved C6 1.19 mm to (117.4, 120.5)
- moved C7 1.19 mm to (157.8, 108.0)
- moved ESC1 1.19 mm to (131.1, 108.0)
- moved ESC_DEBUG1 1.19 mm to (123.2, 106.8)
- moved H1 1.19 mm to (160.7, 113.2)
- moved H2 1.19 mm to (115.7, 126.2)
- moved Q1 1.19 mm to (125.0, 121.4)
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Connections:
- XIAO_L1 pad 2: Net-(ESC1-Pin_7) -> Net-(SPI1-Pin_3)
- XIAO_L1 pad 3: Net-(ESC1-Pin_6) -> Net-(ESC1-Pin_7)
- XIAO_L1 pad 4: Net-(ESC1-Pin_5) -> Net-(ESC1-Pin_6)
- XIAO_L1 pad 5: Net-(ESC1-Pin_4) -> Net-(ESC1-Pin_5)
- XIAO_L1 pad 6: VSENSE -> Net-(ESC1-Pin_4)
- XIAO_L1 pad 7: Net-(SPI1-Pin_4) -> VSENSE
- XIAO_R1 pad 4: Net-(SPI1-Pin_2) -> Net-(SPI1-Pin_4)
- XIAO_R1 pad 6: Net-(SPI1-Pin_3) -> Net-(SPI1-Pin_2)
Routing:
- net Net-(SPI1-Pin_3): track 12.4 -> 24.7 mm
- net Net-(SPI1-Pin_2): track 19.8 -> 16.9 mm
- net Net-(SPI1-Pin_4): track 20.5 -> 22.7 mm
- net VSENSE: track 11.9 -> 14.0 mm
- net Net-(ESC1-Pin_5): track 24.6 -> 26.4 mm
- net Net-(ESC1-Pin_4): track 14.3 -> 15.9 mm
- net Net-(ESC1-Pin_6): track 22.3 -> 23.4 mm
- net Net-(ESC1-Pin_7): track 28.1 -> 27.1 mm
- net Net-(SPI1-Pin_1): track 14.3 -> 13.6 mm
- added copper zone on F.Cu, net (none)
Other:
- board text added: "Drone Motherboard V1.1"
- board text removed: "Drone Motherboard V1"

Commit message: Make v in version silkscreen lowercase
Other:
- board text added: "Drone Motherboard v1.1"
- board text removed: "Drone Motherboard V1.1"
Changed lines of the file:
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@@
 		)
 	)
-	(gr_text "Drone Motherboard V1.1"
+	(gr_text "Drone Motherboard v1.1"
 		(at 113.5 122.2 0)
 		(layer "B.SilkS")

Commit message: Replace telemetry with VBat sense
Parts:
- added C7: 0.1u, Capacitor_SMD:C_0603_1608Metric_Pad1.08x0.95mm_HandSolder, F.Cu at (129.6, 112.8)
- added R3: 33k, Resistor_SMD:R_0603_1608Metric_Pad0.98x0.95mm_HandSolder, F.Cu at (126.0, 112.8)
- added R4: 8.2k, Resistor_SMD:R_0603_1608Metric_Pad0.98x0.95mm_HandSolder, F.Cu at (127.8, 112.8)
- renumbered C7 to C8
Connections:
- ESC1 pad 1: unconnected-(ESC1-Pin_1-Pad1) -> Net-(ESC1-Pin_1)
- ESC1 pad 2: Net-(ESC1-Pin_2) -> unconnected-(ESC1-Pin_2-Pad2)
- ESC_DEBUG1 pad 5: Net-(ESC1-Pin_2) -> Net-(ESC1-Pin_1)
- XIAO_R1 pad 7: Net-(ESC1-Pin_2) -> Net-(XIAO_R1-Pin_7)
Routing:
- net Net-(ESC1-Pin_2): track 50.0 -> 0.00 mm, vias 1 -> 0
- net Net-(XIAO_R1-Pin_7): track 0.00 -> 35.2 mm, vias 0 -> 1
- net Net-(ESC1-Pin_1): track 0.00 -> 15.8 mm
- net GND: track 3.91 -> 1.16 mm, vias 32 -> 34
- removed copper zone on F.Cu, net (none)
Other:
- board text added: "VBAT"
- board text removed: "TLM"
